Commit message: removed collisions from goal. fixed goal distance

File: src/arm_description/urdf/arm_gazebo.urdf (robot description, URDF)
Before this commit: robot arm, 9 links, 8 joints
Joints:
- joint eef_joint: origin (none) -> xyz=0 0 0.120 rpy=0 0 0

File: src/arm_description/urdf/ball.urdf (robot description, URDF)
Before this commit: robot simple_ball, 1 links, 0 joints
Links:
- link ball: geometry visual sphere radius=0.07
