Commit message: started training with ddpg algo

File: src/arm_description/urdf/ball.urdf (robot description, URDF)
Before this commit: robot simple_ball, 1 links, 0 joints
Links:
- link ball: geometry visual sphere radius=0.05

Commit message: modified reward structure. increased goal radius

File: src/arm_description/urdf/ball.urdf (robot description, URDF)
Before this commit: robot simple_ball, 1 links, 0 joints
Links:
- link ball: geometry visual sphere radius=0.06
